File: design.kicad_pcb (KiCad board)
At the start: 2 copper layers, 53 x 26.2 mm, 0 parts

Commit message: update
Parts:
- added J1: 2601-3108, Snapeda:CONN8_2601-3108_WAG, F.Cu at (140.0, 115.1)
- added J2: 2601-3108, Snapeda:CONN8_2601-3108_WAG, F.Cu at (99.0, 75.6)
- added J3: 2601-3108, Snapeda:CONN8_2601-3108_WAG, F.Cu at (131.4, 75.6)
- added U1: ATtiny1616-S, Package_SO:SOIC-20W_7.5x12.8mm_P1.27mm, F.Cu at (126.2, 94.6)
Other:
- board size 53 x 26.2 mm -> 79 x 55 mm

Commit message: update
Parts:
- added C1: 1uF, Capacitor_SMD:C_0805_2012Metric, F.Cu at (95.0, 103.2)
- added C2: 1uF, Capacitor_SMD:C_0805_2012Metric, F.Cu at (121.7, 86.0)
- added D1: 5V, LED_SMD:LED_0805_2012Metric, F.Cu at (99.5, 103.2)
- added D2: 3.3V, LED_SMD:LED_0805_2012Metric, F.Cu at (109.9, 96.5)
- added D3: 5V, LED_SMD:LED_0805_2012Metric, F.Cu at (116.6, 90.4)
- added D4: 3.3V, LED_SMD:LED_0805_2012Metric, F.Cu at (103.9, 103.2)
- added J4: TYPE-C-31-M-12, Snapeda:TYPE-C-31-M-12_HRO_TYPE-C-31-M-12, F.Cu at (89.6, 87.4)
- added J5: SKEDD-UPDI-4, Connector_custom:SKEDD-UPDI-4, F.Cu at (93.0, 103.3)
- added R1: 5.1k, Resistor_SMD:R_0805_2012Metric, F.Cu at (116.6, 93.4)
- added R2: 5.1k, Resistor_SMD:R_0805_2012Metric, F.Cu at (114.3, 100.5)
- added R3: 330, Resistor_SMD:R_0805_2012Metric, F.Cu at (126.2, 86.0)
- added R4: 330, Resistor_SMD:R_0805_2012Metric, F.Cu at (121.7, 89.0)
- added R5: 330, Resistor_SMD:R_0805_2012Metric, F.Cu at (121.0, 91.9)
- added R6: 330, Resistor_SMD:R_0805_2012Metric, F.Cu at (108.3, 103.5)
- added S1: JS202011JCQN, Snapeda:SW_JS202011JCQN, F.Cu at (111.6, 89.8)
- added U2: AP2112K-3.3, Package_TO_SOT_SMD:SOT-23-5, F.Cu at (116.9, 86.7)
- added U3: LM73100RPWR, Snapeda:LM73100RPWR_IC_LM73100RPWR, F.Cu at (114.6, 97.0)
- added U4: LM73100RPWR, Snapeda:LM73100RPWR_IC_LM73100RPWR, F.Cu at (110.1, 100.0)
- moved J1 23.2 mm to (163.2, 115.0)
- moved J2 10.5 mm to (108.5, 71.2)
- moved J3 9.13 mm to (139.4, 71.2)
- moved U1 6.87 mm to (133.0, 93.6)

Commit message: many changes
Parts:
- removed J2: 2601-3108, Snapeda:CONN8_2601-3108_WAG
- removed U3, U4: LM73100RPWR, Snapeda:LM73100RPWR_IC_LM73100RPWR
- added C3: 0.1uF, Capacitor_SMD:C_0805_2012Metric, F.Cu at (124.5, 91.0)
- added C4: 10uF, Capacitor_SMD:C_0805_2012Metric, F.Cu at (124.5, 95.5)
- added D5: LED1, LED_SMD:LED_0805_2012Metric, F.Cu at (150.9, 95.6)
- added D6: LED2, LED_SMD:LED_0805_2012Metric, F.Cu at (150.8, 98.8)
- added JP1: SolderJumper_2_Bridged, Jumper:SolderJumper-2_P1.3mm_Bridged_Pad1.0x1.5mm, F.Cu at (145.2, 88.0)
- added JP2: SolderJumper_2_Bridged, Jumper:SolderJumper-2_P1.3mm_Bridged_Pad1.0x1.5mm, F.Cu at (146.0, 95.6)
- added JP3: SolderJumper_2_Bridged, Jumper:SolderJumper-2_P1.3mm_Bridged_Pad1.0x1.5mm, F.Cu at (146.0, 98.8)
- added LED1: WS2812B-2020, Snapeda:WS2812B2020, F.Cu at (154.7, 90.6)
- added LED2: WS2812B-2020, Snapeda:WS2812B2020, F.Cu at (151.0, 88.0)
- added LED3: WS2812B-2020, Snapeda:WS2812B2020, F.Cu at (151.0, 90.6)
- added LED4: WS2812B-2020, Snapeda:WS2812B2020, F.Cu at (154.7, 88.0)
- added R7: 330, Resistor_SMD:R_0805_2012Metric, F.Cu at (155.3, 95.6)
- added R8: 330, Resistor_SMD:R_0805_2012Metric, F.Cu at (155.2, 98.8)
- added S2: JS202011JCQN, Snapeda:SW_JS202011JCQN, F.Cu at (93.0, 74.2)
- moved J5 34.1 mm to (104.9, 71.4), turned to 180 degrees
- moved R5 33.5 mm to (98.4, 116.7), turned to 90 degrees
- moved R3 31.7 mm to (97.6, 99.5), turned to -90 degrees
- moved J1 30.9 mm to (132.3, 115.1)
- moved R4 29.6 mm to (94.1, 99.6), turned to -90 degrees
- moved D3 28.9 mm to (98.4, 112.8), turned to -90 degrees
- moved R1 26.7 mm to (92.9, 81.1), turned to 180 degrees
- moved R2 22.4 mm to (93.0, 93.7)
- moved C2 20.8 mm to (101.0, 84.0), turned to 180 degrees
- moved R6 20.0 mm to (93.3, 116.7), turned to 90 degrees
- moved J3 17.3 mm to (122.2, 71.1)
- moved D2 17.2 mm to (94.1, 103.4), turned to 90 degrees
- moved U2 16.0 mm to (101.0, 88.1)
- moved D4 14.3 mm to (93.3, 112.8), turned to -90 degrees
- moved C1 12.5 mm to (101.0, 92.2)
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Connections:
- J1 pad 1: unconnected-(J1-Pad1) -> PA7
- J1 pad 10: unconnected-(J1-Pad10) -> GND
- J1 pad 11: unconnected-(J1-Pad11) -> GND
- J1 pad 12: unconnected-(J1-Pad12) -> GND
- J1 pad 13: unconnected-(J1-Pad13) -> VDD
- J1 pad 14: unconnected-(J1-Pad14) -> VDD
- J1 pad 15: unconnected-(J1-Pad15) -> VBUS
- J1 pad 16: unconnected-(J1-Pad16) -> VBUS
- J1 pad 2: unconnected-(J1-Pad2) -> PA7
- J1 pad 3: unconnected-(J1-Pad3) -> PA6
- J1 pad 4: unconnected-(J1-Pad4) -> PA6
- J1 pad 5: unconnected-(J1-Pad5) -> PA5
- J1 pad 6: unconnected-(J1-Pad6) -> PA5
- J1 pad 7: unconnected-(J1-Pad7) -> PA4
- J1 pad 8: unconnected-(J1-Pad8) -> PA4
- J1 pad 9: unconnected-(J1-Pad9) -> GND
- J3 pad 1: unconnected-(J3-Pad1) -> PA3
- J3 pad 10: unconnected-(J3-Pad10) -> PC3
- J3 pad 11: unconnected-(J3-Pad11) -> PC2
- J3 pad 12: unconnected-(J3-Pad12) -> PC2
- J3 pad 13: unconnected-(J3-Pad13) -> PC1
- J3 pad 14: unconnected-(J3-Pad14) -> PC1
- J3 pad 15: unconnected-(J3-Pad15) -> PC0
- J3 pad 16: unconnected-(J3-Pad16) -> PC0
- J3 pad 2: unconnected-(J3-Pad2) -> PA3
- J3 pad 3: unconnected-(J3-Pad3) -> PA2
- J3 pad 4: unconnected-(J3-Pad4) -> PA2
- J3 pad 5: unconnected-(J3-Pad5) -> PA1
- J3 pad 6: unconnected-(J3-Pad6) -> PA1
- J3 pad 7: unconnected-(J3-Pad7) -> PA0
- J3 pad 8: unconnected-(J3-Pad8) -> PA0
- J3 pad 9: unconnected-(J3-Pad9) -> PC3
- J4 pad A6: D+ -> unconnected-(J4-PadA6)
- J4 pad A7: D- -> unconnected-(J4-PadA7)
- J4 pad B6: D+ -> unconnected-(J4-PadB6)
- J4 pad B7: D- -> unconnected-(J4-PadB7)
- R3 pad 1: VBUS -> V_switch
- R5 pad 1: VBUS -> V_switch
- S1 pad 1: VBUS -> unconnected-(S1-Pad1)
- U1 pad 1: unconnected-(U1-Pad1) -> VDD
- U1 pad 10: unconnected-(U1-Pad10) -> PB1
- U1 pad 11: unconnected-(U1-Pad11) -> PB0
- U1 pad 12: unconnected-(U1-Pad12) -> PC0
- U1 pad 13: unconnected-(U1-Pad13) -> PC1
- U1 pad 14: unconnected-(U1-Pad14) -> PC2
- U1 pad 15: unconnected-(U1-Pad15) -> PC3
- U1 pad 16: unconnected-(U1-Pad16) -> PA0
- U1 pad 17: unconnected-(U1-Pad17) -> PA1
- U1 pad 18: unconnected-(U1-Pad18) -> PA2
- U1 pad 19: unconnected-(U1-Pad19) -> PA3
- U1 pad 2: unconnected-(U1-Pad2) -> PA4
- U1 pad 20: unconnected-(U1-Pad20) -> GND
- U1 pad 3: unconnected-(U1-Pad3) -> PA5
- U1 pad 4: unconnected-(U1-Pad4) -> PA6
- U1 pad 5: unconnected-(U1-Pad5) -> PA7
- U1 pad 6: unconnected-(U1-Pad6) -> PB5
- U1 pad 7: unconnected-(U1-Pad7) -> PB4
- U1 pad 8: unconnected-(U1-Pad8) -> PB3
- U1 pad 9: unconnected-(U1-Pad9) -> PB2

Commit message: update
Parts:
- added J2: 2601-3108, Snapeda:CONN8_2601-3108_WAG, F.Cu at (163.2, 114.9)
- moved LED3 4.75 mm to (155.0, 88.0)
- moved LED1 4.54 mm to (151.0, 88.0)
- moved LED4 2.99 mm to (155.0, 91.0)
- moved LED2 2.98 mm to (151.0, 91.0)
- moved D2 2.95 mm to (93.3, 106.3)
- moved D1 2.94 mm to (98.4, 106.3)
- moved J3 1.35 mm to (120.8, 71.1)
- moved R4 1.32 mm to (93.3, 100.6)
- moved R3 1.31 mm to (98.4, 100.6)
- moved R2 1.30 mm to (93.0, 95.0)
- moved C1 1.22 mm to (101.0, 91.0)
- moved R5 1.06 mm to (98.4, 117.7)
- moved R6 1.06 mm to (93.3, 117.7)
- moved C2 1.05 mm to (101.0, 85.0)
- moved J4 0.85 mm to (89.0, 88.0)
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Connections:
- C1 pad 1: VBUS -> V_switch
- S1 pad 1: unconnected-(S1-Pad1) -> V_switch
- U2 pad 1: VBUS -> V_switch
- U2 pad 3: VBUS -> V_switch

Commit message: lot of updates
Parts:
- moved S2 13.3 mm to (105.0, 80.0), turned to -90 degrees
- moved R6 6.40 mm to (99.0, 114.8)
- moved D4 6.02 mm to (99.0, 110.1)
- moved C1 5.98 mm to (101.0, 85.0)
- moved D2 5.86 mm to (99.0, 105.0)
- moved R5 5.83 mm to (93.3, 114.8)
- moved R4 5.72 mm to (99.0, 100.6)
- moved D3 5.42 mm to (93.3, 110.1)
- moved D1 5.23 mm to (93.3, 105.0)
- moved R3 5.08 mm to (93.3, 100.6)
- moved C2 5.00 mm to (105.0, 88.0), turned to -90 degrees
- moved LED1 1.45 mm to (151.0, 86.5)
- moved LED2 1.45 mm to (151.0, 89.5)
- moved LED3 1.45 mm to (155.0, 86.5)
- moved LED4 1.45 mm to (155.0, 89.5)
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Connections:
- J5 pad 3: UPDI -> PA0
- J5 pad 4: TX -> PA1
Routing:
- net VDD: track 0.00 -> 115.8 mm
- net VBUS: track 0.00 -> 61.5 mm
- net PA0: track 0.00 -> 48.5 mm
- net V_switch: track 0.00 -> 47.2 mm
- net PB0: track 0.00 -> 46.7 mm
- net Net-(S1-Pad5): track 0.00 -> 46.1 mm
- net +3V3: track 0.00 -> 43.9 mm
- net PA1: track 0.00 -> 41.0 mm
- net PB1: track 0.00 -> 40.8 mm
- net PB2: track 0.00 -> 32.8 mm
- net PB3: track 0.00 -> 28.8 mm
- net PB4: track 0.00 -> 25.5 mm
- net PB5: track 0.00 -> 24.6 mm
- net PC0: track 0.00 -> 20.5 mm
- net PA3: track 0.00 -> 20.5 mm
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- added copper zone on B.Cu, net GND
- added copper zone on F.Cu, net GND
- added copper zone on F.Cu, net VBUS
- added copper zone on F.Cu, net VDD
- added copper zone on F.Cu, net V_switch

Commit message: update edge layer
Routing:
- net VBUS: track 61.5 -> 65.7 mm
Other:
- board size 79 x 55 mm -> 80 x 55 mm
Changed lines of the file:
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@@
     )
   )
-  (gr_rect (start 87.5 65.6) (end 166.5 120.6) (layer "Edge.Cuts") (width 0.05) (fill none))
+  (gr_rect (start 87.5 65.75) (end 167.5 120.75) (layer "Edge.Cuts") (width 0.05) (fill none))
   (gr_text "<<project_name>>\n<<ID>>\n<<version>>\n<<date>>\n<<hash>>\n<<website_link>>" (at 225.75 151) (layer "F.SilkS")
     (effects (font (size 1 1) (thickness 0.15)))
   )
-  (dimension (type aligned) (layer "Edge.Cuts")
-    (pts (xy 87.5 65.6) (xy 166.5 65.6))
+  (dimension (type aligned) (layer "Dwgs.User")
+    (pts (xy 87.5 65.75) (xy 167.5 65.75))
     (height -3.65)
-    (gr_text "79,0000 mm" (at 127 60.8) (layer "Edge.Cuts")
+    (gr_text "80,0000 mm" (at 127.5 60.95) (layer "Dwgs.User")
       (effects (font (size 1 1) (thickness 0.15)))
     )
     (format (units 3) (units_format 1) (precision 4))
     (style (thickness 0.05) (arrow_length 1.27) (text_position_mode 0) (extension_height 0.58642) (extension_offset 0.5) keep_text_aligned)
+  )
+  (dimension (type aligned) (layer "Dwgs.User")
+    (pts (xy 167.5 65.75) (xy 167.5 120.75))
+    (height -3.909491)
+    (gr_text "55,0000 mm" (at 170.259491 93.25 90) (layer "Dwgs.User")
+      (effects (font (size 1 1) (thickness 0.15)))
+    )
+    (format (units 3) (units_format 1) (precision 4))
+    (style (thickness 0.1) (arrow_length 1.27) (text_position_mode 0) (extension_height 0.58642) (extension_offset 0.5) keep_text_aligned)
   )
   (segment (start 146.66 95) (end 150.0625 95) (width 0.21) (layer "F.Cu") (net 1))
@@
   (segment (start 107.695096 117.554904) (end 105.75 119.5) (width 0.5) (layer "F.Cu") (net 33))
   (segment (start 105.75 119.5) (end 91 119.5) (width 0.5) (layer "F.Cu") (net 33))
+  (segment (start 93.75 90.4) (end 95.6 90.4) (width 0.5) (layer "F.Cu") (net 33))
+  (segment (start 95.35 85.6) (end 95.75 86) (width 0.5) (layer "F.Cu") (net 33))
   (segment (start 96 97.5) (end 97.75 95.75) (width 0.5) (layer "F.Cu") (net 33))
   (segment (start 91 119.5) (end 89.75 118.25) (width 0.5) (layer "F.Cu") (net 33))
@@
   (segment (start 107.695096 114.695096) (end 107.695096 109.885001) (width 0.5) (layer "F.Cu") (net 33))
   (segment (start 107.695096 114.885001) (end 107.695096 117.554904) (width 0.5) (layer "F.Cu") (net 33))
+  (segment (start 95.6 90.4) (end 95.75 90.25) (width 0.5) (layer "F.Cu") (net 33))
   (segment (start 89.75 118.25) (end 89.75 99.5) (width 0.5) (layer "F.Cu") (net 33))
+  (segment (start 93.75 85.6) (end 95.35 85.6) (width 0.5) (layer "F.Cu") (net 33))
   (segment (start 107.885001 114.885001) (end 107.695096 114.695096) (width 0.5) (layer "F.Cu") (net 33))
   (segment (start 99.8625 88) (end 98 88) (width 0.5) (layer "F.Cu") (net 34))
@@
     (polygon
       (pts
-        (xy 107 83)
+        (xy 106.5 83)
         (xy 116 83)
         (xy 116 93)
@@
         (xy 111 90)
         (xy 107 86)
-        (xy 103 86)
-        (xy 103 77)
-        (xy 107 77)
+        (xy 103.5 86)
+        (xy 103.5 77)
+        (xy 106.5 77)
       )
     )
@@
       (pts
         (xy 116 96)
-        (xy 116 96)
-        (xy 116 90)
+        (xy 116.5 96)
+        (xy 116.5 90)
         (xy 128 90)
         (xy 128 100)

Commit message: Update design.kicad_pcb
Routing:
- net GND: vias 52 -> 48
Other:
- outline, holes or cut-outs redrawn
Changed lines of the file:
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@@
     )
   )
-  (gr_rect (start 87.5 65.75) (end 167.5 120.75) (layer "Edge.Cuts") (width 0.05) (fill none))
-  (gr_text "<<project_name>>\n<<ID>>\n<<version>>\n<<date>>\n<<hash>>\n<<website_link>>" (at 225.75 151) (layer "F.SilkS")
+  (gr_arc (start 87.5 68.25) (mid 88.232233 66.482233) (end 90 65.75) (layer "Edge.Cuts") (width 0.05))
+  (gr_line (start 90 65.75) (end 165 65.75) (layer "Edge.Cuts") (width 0.05))
+  (gr_arc (start 90 120.75) (mid 88.232233 120.017767) (end 87.5 118.25) (layer "Edge.Cuts") (width 0.05))
+  (gr_line (start 167.5 68.25) (end 167.5 118.25) (layer "Edge.Cuts") (width 0.05))
+  (gr_line (start 165 120.75) (end 90 120.75) (layer "Edge.Cuts") (width 0.05))
+  (gr_arc (start 165 65.75) (mid 166.767767 66.482233) (end 167.5 68.25) (layer "Edge.Cuts") (width 0.05))
+  (gr_arc (start 167.5 118.25) (mid 166.767767 120.017767) (end 165 120.75) (layer "Edge.Cuts") (width 0.05))
+  (gr_line (start 87.5 118.25) (end 87.5 68.25) (layer "Edge.Cuts") (width 0.05))
+  (gr_text "<<project_name>>\n<<ID>>\n<<version>>\n<<date>>\n<<hash>>\n<<website_link>>" (at 133 92.75) (layer "B.SilkS")
     (effects (font (size 1 1) (thickness 0.15)))
   )
@@
   (via (at 126.75 112.5) (size 0.8) (drill 0.4) (layers "F.Cu" "B.Cu") (free) (net 34))
   (via (at 95.25 107.75) (size 0.8) (drill 0.4) (layers "F.Cu" "B.Cu") (free) (net 34))
-  (via (at 137.75 93.75) (size 0.8) (drill 0.4) (layers "F.Cu" "B.Cu") (free) (net 34))
   (via (at 151.75 84.25) (size 0.8) (drill 0.4) (layers "F.Cu" "B.Cu") (free) (net 34))
   (via (at 151.75 80.5) (size 0.8) (drill 0.4) (layers "F.Cu" "B.Cu") (free) (net 34))
@@
   (via (at 95.75 92.25) (size 0.8) (drill 0.4) (layers "F.Cu" "B.Cu") (net 34))
   (via (at 125 86.75) (size 0.8) (drill 0.4) (layers "F.Cu" "B.Cu") (free) (net 34))
-  (via (at 131 91.75) (size 0.8) (drill 0.4) (layers "F.Cu" "B.Cu") (free) (net 34))
   (via (at 89.25 89) (size 0.8) (drill 0.4) (layers "F.Cu" "B.Cu") (free) (net 34))
   (via (at 122.5 78) (size 0.8) (drill 0.4) (layers "F.Cu" "B.Cu") (free) (net 34))
@@
   (via (at 89.25 80.5) (size 0.8) (drill 0.4) (layers "F.Cu" "B.Cu") (free) (net 34))
   (via (at 123.5 112.5) (size 0.8) (drill 0.4) (layers "F.Cu" "B.Cu") (free) (net 34))
-  (via (at 131 94) (size 0.8) (drill 0.4) (layers "F.Cu" "B.Cu") (free) (net 34))
-  (via (at 137.75 91.75) (size 0.8) (drill 0.4) (layers "F.Cu" "B.Cu") (free) (net 34))
   (via (at 103.25 91.75) (size 0.8) (drill 0.4) (layers "F.Cu" "B.Cu") (free) (net 34))
   (via (at 115.25 76) (size 0.8) (drill 0.4) (layers "F.Cu" "B.Cu") (free) (net 34))

Commit message: update
Parts:
- moved LED2 5.03 mm to (155.0, 86.5)
- moved LED3 4.97 mm to (151.0, 89.5)
Connections:
- LED2 pad 1: Net-(LED2-Pad1) -> Net-(LED3-Pad3)
- LED2 pad 3: Net-(LED2-Pad3) -> Net-(LED1-Pad1)
- LED3 pad 1: Net-(LED2-Pad3) -> Net-(LED3-Pad1)
- LED3 pad 3: Net-(LED1-Pad1) -> Net-(LED3-Pad3)
- LED4 pad 3: Net-(LED2-Pad1) -> Net-(LED3-Pad1)
Routing:
- net Net-(LED3-Pad3): track 0.00 -> 6.97 mm
- net Net-(LED2-Pad3): track 6.97 -> 0.00 mm
- net Net-(LED3-Pad1): track 0.00 -> 2.77 mm
- net Net-(LED2-Pad1): track 2.77 -> 0.00 mm
- net GND: track 16.1 -> 15.8 mm, vias 48 -> 59
Other:
- board text added: "3.3V"
- board text added: "5V"
- board text added: "ATtiny 416/816/1616/3216"
- board text added: "D/A PA7"
- board text added: "D/A PB4"
- board text added: "D/A PB5"
- board text added: "D/A ⎍ PA6"
- board text added: "D/A 〜 PA4"
- board text added: "D/A 〜 PA5"
- board text added: "GND"
- board text added: "In 1.8V-5V WS2812 5V"
- board text added: "PA0 D/A UPDI"
- board text added: "PA1 D/A"
- board text added: "PA2 ⎍ D/A"
- board text added: "PA3 〜 D/A"
- board text added: "PB1"
- board text added: "PB2"
- board text added: "PC0 〜 D"
- board text added: "PC1 〜 D"
- board text added: "PC2 ⎍ D"
- board text added: "PC3 D"
- board text added: "Power Rail Status"
- board text added: "RX D PB3"
- board text added: "SCL D/A 〜 PB0"
- board text added: "SDA D/A 〜 PB1"
- board text added: "Selected Volatge"
- board text added: "TX D 〜⎍ PB2"
- board text added: "UPDI"
- board text added: "USB"
- board text added: "VBUS"
- board text added: "VDD"
- board text added: "⎍ Async Interrrupt 〜 PWM D/A Digital/Analog"
