File: USB2UART.kicad_sch (KiCad schematic)
At the start: 14 parts

Commit message: remove subsheet USB2UART
Parts:
- removed C? (x2): 1uF, symbol Device:C_Small
- removed C?: 0.1uF, symbol Device:C_Small
- removed D? (x4): Red, symbol Device:LED_Small
- removed R?: 1k, symbol Device:R_Small
- removed R? (x4): 220, symbol Device:R_Small
- removed R?: 4.7k, symbol Device:R_Small
- removed U?: CP2105, Snapeda:CP2105_QFN24_0.5, symbol Snapeda:CP2105
Connections:
- no-connect marks 8 -> 0
Other:
- note removed: "PA1 TX_MCU PA2 RX_MCU"
