File: design.kicad_sch (KiCad schematic)
At the start: 80 parts, among them J1 2601-3108, J10 Conn_01x04, J11 Conn_01x04, J12 Conn_01x03, J13 Conn_01x03, J14 Conn_01x04, J2 2601-3108, J3 2601-3108, J4 TYPE-C-31-M-12, J5 SKEDD-UPDI-4, J6 Conn_01x04, J7 Conn_01x04, J8 Conn_01x04, J9 Conn_01x04, U1 ATtiny1616-S, U2 AP2112K-3.3, U3 CP2105

Commit message: many updates
Parts:
- removed D7: Red, LED_SMD:LED_0805_2012Metric, symbol Device:LED_Small
- removed R11: 220, Resistor_SMD:R_0805_2012Metric, symbol Device:R_Small
Connections:
- net PA1: no longer J5.4 (TX_MCU), U3.20 (RXD_SCI)
- net PA2: no longer U3.21 (TXD_SCI)
- net PB2: now also J5.4 (TX_MCU), U3.20 (RXD_SCI)
- net PB3: now also U3.21 (TXD_SCI)
- no-connect marks 12 -> 13
Changed lines of the file:
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@@
   (junction (at 21.717 170.18) (diameter 0) (color 0 0 0 0)
   )
-  (junction (at 274.32 205.74) (diameter 0) (color 0 0 0 0)
-  )
   (junction (at 21.717 172.72) (diameter 0) (color 0 0 0 0)
   )
@@
   (no_connect (at 248.92 233.68))
   (no_connect (at 68.58 45.72))
+  (no_connect (at 248.92 226.06))
   (no_connect (at 248.92 256.54))
   (no_connect (at 248.92 251.46))
@@
     (stroke (width 0) (type default) (color 0 0 0 0))
   )
-  (wire (pts (xy 269.24 205.74) (xy 269.24 208.28))
-    (stroke (width 0) (type default) (color 0 0 0 0))
-  )
   (wire (pts (xy 383.54 106.68) (xy 325.12 106.68))
     (stroke (width 0) (type default) (color 0 0 0 0))
@@
     (stroke (width 0) (type default) (color 0 0 0 0))
   )
-  (wire (pts (xy 274.32 203.2) (xy 274.32 205.74))
+  (wire (pts (xy 279.4 203.2) (xy 279.4 208.28))
     (stroke (width 0) (type default) (color 0 0 0 0))
   )
@@
     (stroke (width 0) (type default) (color 0 0 0 0))
   )
-  (wire (pts (xy 269.24 213.36) (xy 269.24 218.44))
-    (stroke (width 0) (type default) (color 0 0 0 0))
-  )
   (wire (pts (xy 106.68 48.641) (xy 116.078 48.641))
     (stroke (width 0) (type default) (color 0 0 0 0))
@@
     (stroke (width 0) (type default) (color 0 0 0 0))
   )
-  (wire (pts (xy 274.32 205.74) (xy 269.24 205.74))
-    (stroke (width 0) (type default) (color 0 0 0 0))
-  )
   (wire (pts (xy 59.69 228.6) (xy 66.04 228.6))
     (stroke (width 0) (type default) (color 0 0 0 0))
@@
     (stroke (width 0) (type default) (color 0 0 0 0))
   )
-  (wire (pts (xy 269.24 226.06) (xy 248.92 226.06))
-    (stroke (width 0) (type default) (color 0 0 0 0))
-  )
   (wire (pts (xy 353.06 160.02) (xy 353.06 157.48))
     (stroke (width 0) (type default) (color 0 0 0 0))
@@
     (stroke (width 0) (type default) (color 0 0 0 0))
   )
-  (wire (pts (xy 269.24 223.52) (xy 269.24 226.06))
-    (stroke (width 0) (type default) (color 0 0 0 0))
-  )
   (wire (pts (xy 74.295 48.26) (xy 68.58 48.26))
     (stroke (width 0) (type default) (color 0 0 0 0))
@@
     (stroke (width 0) (type default) (color 0 0 0 0))
   )
-  (wire (pts (xy 279.4 208.28) (xy 279.4 205.74))
-    (stroke (width 0) (type default) (color 0 0 0 0))
-  )
   (wire (pts (xy 73.66 182.88) (xy 71.12 182.88))
     (stroke (width 0) (type default) (color 0 0 0 0))
@@
     (stroke (width 0) (type default) (color 0 0 0 0))
   )
-  (wire (pts (xy 274.32 205.74) (xy 279.4 205.74))
-    (stroke (width 0) (type default) (color 0 0 0 0))
-  )
   (wire (pts (xy 73.66 149.86) (xy 73.66 152.4))
     (stroke (width 0) (type default) (color 0 0 0 0))
@@
     )
   )
+  (global_label "PB2" (shape input) (at 266.7 157.48 0) (fields_autoplaced)
+    (effects (font (size 1.27 1.27)) (justify left))
+    (property "Referenzen zwischen Schaltplänen" "${INTERSHEET_REFS}" (id 0) (at 272.7737 157.4006 0)
+      (effects (font (size 1.27 1.27)) (justify left) hide)
+    )
+  )
   (global_label "PA1" (shape input) (at 91.44 81.28 0) (fields_autoplaced)
     (effects (font (size 1.27 1.27)) (justify left))
@@
     )
   )
-  (global_label "PA1" (shape input) (at 266.7 157.48 0) (fields_autoplaced)
-    (effects (font (size 1.27 1.27)) (justify left))
-    (property "Referenzen zwischen Schaltplänen" "${INTERSHEET_REFS}" (id 0) (at 272.5923 157.4006 0)
-      (effects (font (size 1.27 1.27)) (justify left) hide)
-    )
-  )
   (global_label "VBUS" (shape input) (at 203.2 231.14 180) (fields_autoplaced)
     (effects (font (size 1.27 1.27)) (justify right))
@@
     )
   )
+  (global_label "PB3" (shape input) (at 248.92 248.92 0) (fields_autoplaced)
+    (effects (font (size 1.27 1.27)) (justify left))
+    (property "Referenzen zwischen Schaltplänen" "${INTERSHEET_REFS}" (id 0) (at 254.9937 248.8406 0)
+      (effects (font (size 1.27 1.27)) (justify left) hide)
+    )
+  )
   (global_label "PC0" (shape input) (at 60.96 101.6 180) (fields_autoplaced)
     (effects (font (size 1.27 1.27)) (justify right))
@@
     )
   )
-  (global_label "VIO" (shape input) (at 274.32 203.2 90) (fields_autoplaced)
+  (global_label "VIO" (shape input) (at 279.4 203.2 90) (fields_autoplaced)
     (effects (font (size 1.27 1.27)) (justify left))
-    (property "Referenzen zwischen Schaltplänen" "${INTERSHEET_REFS}" (id 0) (at 274.3994 197.852 90)
+    (property "Referenzen zwischen Schaltplänen" "${INTERSHEET_REFS}" (id 0) (at 279.4794 197.852 90)
       (effects (font (size 1.27 1.27)) (justify left) hide)
     )
@@
     )
   )
+  (global_label "PB2" (shape input) (at 248.92 246.38 0) (fields_autoplaced)
+    (effects (font (size 1.27 1.27)) (justify left))
+    (property "Referenzen zwischen Schaltplänen" "${INTERSHEET_REFS}" (id 0) (at 254.9937 246.3006 0)
+      (effects (font (size 1.27 1.27)) (justify left) hide)
+    )
+  )
   (global_label "VIO" (shape input) (at 198.12 215.9 180) (fields_autoplaced)
     (effects (font (size 1.27 1.27)) (justify right))
@@
     )
   )
-  (global_label "PA1" (shape input) (at 248.92 246.38 0) (fields_autoplaced)
-    (effects (font (size 1.27 1.27)) (justify left))
-    (property "Referenzen zwischen Schaltplänen" "${INTERSHEET_REFS}" (id 0) (at 254.8123 246.3006 0)
-      (effects (font (size 1.27 1.27)) (justify left) hide)
-    )
-  )
   (global_label "D+" (shape input) (at 33.02 35.56 180) (fields_autoplaced)
     (effects (font (size 1.27 1.27)) (justify right))
@@
     )
   )
-  (global_label "PA2" (shape input) (at 248.92 248.92 0) (fields_autoplaced)
-    (effects (font (size 1.27 1.27)) (justify left))
-    (property "Referenzen zwischen Schaltplänen" "${INTERSHEET_REFS}" (id 0) (at 254.8123 248.8406 0)
-      (effects (font (size 1.27 1.27)) (justify left) hide)
-    )
-  )
   (global_label "PB3" (shape input) (at 73.66 165.1 180) (fields_autoplaced)
     (effects (font (size 1.27 1.27)) (justify right))
@@
     (pin "1")
   )
-  (symbol (lib_id "Device:R_Small") (at 269.24 210.82 0) (unit 1)
-    (in_bom yes) (on_board yes) (fields_autoplaced)
-    (property "Reference" "R11" (id 0) (at 271.78 209.5499 0)
-      (effects (font (size 1.27 1.27)) (justify left))
-    )
-    (property "Value" "220" (id 1) (at 271.78 212.0899 0)
-      (effects (font (size 1.27 1.27)) (justify left))
-    )
-    (property "Footprint" "Resistor_SMD:R_0805_2012Metric" (id 2) (at 269.24 210.82 0)
-      (effects (font (size 1.27 1.27)) hide)
-    )
-    (property "Datasheet" "~" (id 3) (at 269.24 210.82 0)
-      (effects (font (size 1.27 1.27)) hide)
-    )
-    (pin "1")
-    (pin "2")
-  )
   (symbol (lib_name "WS2812B-2020_3") (lib_id "Snapeda:WS2812B-2020") (at 325.12 198.12 0) (unit 1)
     (in_bom yes) (on_board yes) (fields_autoplaced)
@@
     (pin "4")
   )
-  (symbol (lib_id "Device:LED_Small") (at 269.24 220.98 90) (unit 1)
-    (in_bom yes) (on_board yes) (fields_autoplaced)
-    (property "Reference" "D7" (id 0) (at 271.78 219.6464 90)
-      (effects (font (size 1.27 1.27)) (justify right))
-    )
-    (property "Value" "Red" (id 1) (at 271.78 222.1864 90)
-      (effects (font (size 1.27 1.27)) (justify right))
-    )
-    (property "Footprint" "LED_SMD:LED_0805_2012Metric" (id 2) (at 269.24 220.98 90)
-      (effects (font (size 1.27 1.27)) hide)
-    )
-    (property "Datasheet" "~" (id 3) (at 269.24 220.98 90)
-      (effects (font (size 1.27 1.27)) hide)
-    )
-    (pin "1")
-    (pin "2")
-  )
   (symbol (lib_id "Device:R_Small") (at 279.4 210.82 0) (unit 1)
     (in_bom yes) (on_board yes) (fields_autoplaced)
@@
       (reference "D6") (unit 1) (value "LED2") (footprint "LED_SMD:LED_0805_2012Metric")
     )
-    (path "/a7464efb-a4a0-4ffd-bc4f-072fd8d316a1"
-      (reference "D7") (unit 1) (value "Red") (footprint "LED_SMD:LED_0805_2012Metric")
-    )
     (path "/db5ca8c2-4986-41e1-aec1-ef6e7f873716"
       (reference "D8") (unit 1) (value "Red") (footprint "LED_SMD:LED_0805_2012Metric")
@@
       (reference "R10") (unit 1) (value "4.7k") (footprint "Resistor_SMD:R_0805_2012Metric")
     )
-    (path "/75c1482c-685d-46b0-a20c-d42353437108"
-      (reference "R11") (unit 1) (value "220") (footprint "Resistor_SMD:R_0805_2012Metric")
-    )
     (path "/d3f3b6a4-65f9-4d68-88bb-38ec87453a14"
