File: design.kicad_sch (KiCad schematic)
At the start: 92 parts, among them J1 2601-3108, J10 Conn_01x04, J11 Conn_01x04, J12 Conn_01x03, J13 Conn_01x03, J14 BM04B-SRSS-TB_LF__SN_, J2 2601-3108, J3 2601-3108, J4 TYPE-C-31-M-12, J5 SKEDD-UPDI-4, J6 Conn_01x04, J7 Conn_01x04, J8 Conn_01x04, J9 Conn_01x04, Q1 AO3400A, Q2 AO3400A, SW1 K3-2235S-K1, SW2 K3-2235S-K1, U1 ATtiny1616-S, U2 AP2112K-3.3, U3 CP2105, U4 ATtiny1616-M

Commit message: Update design.kicad_sch
Parts:
- Q1, Q2: JLCPCB (none) -> C20917; LCSC Part (none) -> C20917
- R1, R2: JLCPCB (none) -> C27834; LCSC Part (none) -> C27834
- R10, R11, R15: JLCPCB (none) -> C17673; LCSC Part (none) -> C17673
- R12, R13, R14, R16, R17, R4, R6: JLCPCB (none) -> C17557; LCSC Part (none) -> C17557
- R3, R5, R7, R8: JLCPCB (none) -> C28636; LCSC Part (none) -> C28636
- R9: JLCPCB (none) -> C17513; LCSC Part (none) -> C17513
Changed lines of the file:
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@@
       (effects (font (size 1.27 1.27)) hide)
     )
+    (property "JLCPCB" "C17557" (id 4) (at 152.4 106.68 0)
+      (effects (font (size 1.27 1.27)) hide)
+    )
+    (property "LCSC Part" "C17557" (id 5) (at 152.4 106.68 0)
+      (effects (font (size 1.27 1.27)) hide)
+    )
     (pin "1")
     (pin "2")
@@
       (effects (font (size 1.27 1.27)) hide)
     )
+    (property "JLCPCB" "C17557" (id 4) (at 156.845 40.64 0)
+      (effects (font (size 1.27 1.27)) hide)
+    )
+    (property "LCSC Part" "C17557" (id 5) (at 156.845 40.64 0)
+      (effects (font (size 1.27 1.27)) hide)
+    )
     (pin "1")
     (pin "2")
@@
       (effects (font (size 1.27 1.27)) (justify left) hide)
     )
+    (property "JLCPCB" "C20917" (id 4) (at 203.2 111.76 0)
+      (effects (font (size 1.27 1.27)) hide)
+    )
+    (property "LCSC Part" "C20917" (id 5) (at 203.2 111.76 0)
+      (effects (font (size 1.27 1.27)) hide)
+    )
     (pin "1")
     (pin "2")
@@
       (effects (font (size 1.27 1.27)) hide)
     )
+    (property "JLCPCB" "C17557" (id 4) (at 193.04 106.68 0)
+      (effects (font (size 1.27 1.27)) hide)
+    )
+    (property "LCSC Part" "C17557" (id 5) (at 193.04 106.68 0)
+      (effects (font (size 1.27 1.27)) hide)
+    )
     (pin "1")
     (pin "2")
@@
       (effects (font (size 1.27 1.27)) hide)
     )
+    (property "JLCPCB" "C27834" (id 4) (at 26.035 33.02 0)
+      (effects (font (size 1.27 1.27)) hide)
+    )
+    (property "LCSC Part" "C27834" (id 5) (at 26.035 33.02 0)
+      (effects (font (size 1.27 1.27)) hide)
+    )
     (pin "1")
     (pin "2")
@@
       (effects (font (size 1.27 1.27)) hide)
     )
+    (property "JLCPCB" "C28636" (id 4) (at 165.1 93.98 0)
+      (effects (font (size 1.27 1.27)) hide)
+    )
+    (property "LCSC Part" "C28636" (id 5) (at 165.1 93.98 0)
+      (effects (font (size 1.27 1.27)) hide)
+    )
     (pin "1")
     (pin "2")
@@
       (effects (font (size 1.27 1.27)) hide)
     )
+    (property "JLCPCB" "C28636" (id 4) (at 205.74 93.98 0)
+      (effects (font (size 1.27 1.27)) hide)
+    )
+    (property "LCSC Part" "C28636" (id 5) (at 205.74 93.98 0)
+      (effects (font (size 1.27 1.27)) hide)
+    )
     (pin "1")
     (pin "2")
@@
       (effects (font (size 1.27 1.27)) hide)
     )
+    (property "JLCPCB" "C28636" (id 4) (at 156.845 29.21 0)
+      (effects (font (size 1.27 1.27)) hide)
+    )
+    (property "LCSC Part" "C28636" (id 5) (at 156.845 29.21 0)
+      (effects (font (size 1.27 1.27)) hide)
+    )
     (pin "1")
     (pin "2")
@@
       (effects (font (size 1.27 1.27)) hide)
     )
+    (property "JLCPCB" "C17557" (id 4) (at 279.4 243.84 0)
+      (effects (font (size 1.27 1.27)) hide)
+    )
+    (property "LCSC Part" "C17557" (id 5) (at 279.4 243.84 0)
+      (effects (font (size 1.27 1.27)) hide)
+    )
     (pin "1")
     (pin "2")
@@
       (effects (font (size 1.27 1.27)) hide)
     )
+    (property "JLCPCB" "C17513" (id 4) (at 254 238.76 0)
+      (effects (font (size 1.27 1.27)) hide)
+    )
+    (property "LCSC Part" "C17513" (id 5) (at 254 238.76 0)
+      (effects (font (size 1.27 1.27)) hide)
+    )
     (pin "1")
     (pin "2")
@@
       (effects (font (size 1.27 1.27)) (justify left) hide)
     )
+    (property "JLCPCB" "C20917" (id 4) (at 162.56 111.76 0)
+      (effects (font (size 1.27 1.27)) hide)
+    )
+    (property "LCSC Part" "C20917" (id 5) (at 162.56 111.76 0)
+      (effects (font (size 1.27 1.27)) hide)
+    )
     (pin "1")
     (pin "2")
@@
       (effects (font (size 1.27 1.27)) hide)
     )
+    (property "JLCPCB" "C17557" (id 4) (at 260.35 30.48 0)
+      (effects (font (size 1.27 1.27)) hide)
+    )
+    (property "LCSC Part" "C17557" (id 5) (at 260.35 30.48 0)
+      (effects (font (size 1.27 1.27)) hide)
+    )
     (pin "1")
     (pin "2")
@@
       (effects (font (size 1.27 1.27)) hide)
     )
+    (property "JLCPCB" "C17673" (id 4) (at 256.54 210.82 0)
+      (effects (font (size 1.27 1.27)) hide)
+    )
+    (property "LCSC Part" "C17673" (id 5) (at 256.54 210.82 0)
+      (effects (font (size 1.27 1.27)) hide)
+    )
     (pin "1")
     (pin "2")
@@
       (effects (font (size 1.27 1.27)) hide)
     )
+    (property "JLCPCB" "C17557" (id 4) (at 279.4 210.82 0)
+      (effects (font (size 1.27 1.27)) hide)
+    )
+    (property "LCSC Part" "C17557" (id 5) (at 279.4 210.82 0)
+      (effects (font (size 1.27 1.27)) hide)
+    )
     (pin "1")
     (pin "2")
@@
       (effects (font (size 1.27 1.27)) hide)
     )
+    (property "JLCPCB" "C28636" (id 4) (at 260.35 25.4 0)
+      (effects (font (size 1.27 1.27)) hide)
+    )
+    (property "LCSC Part" "C28636" (id 5) (at 260.35 25.4 0)
+      (effects (font (size 1.27 1.27)) hide)
+    )
     (pin "1")
     (pin "2")
@@
       (effects (font (size 1.27 1.27)) hide)
     )
+    (property "JLCPCB" "C27834" (id 4) (at 77.47 40.64 0)
+      (effects (font (size 1.27 1.27)) hide)
+    )
+    (property "LCSC Part" "C27834" (id 5) (at 77.47 40.64 0)
+      (effects (font (size 1.27 1.27)) hide)
+    )
     (pin "1")
     (pin "2")
@@
       (effects (font (size 1.27 1.27)) hide)
     )
+    (property "JLCPCB" "C17557" (id 4) (at 269.24 243.84 0)
+      (effects (font (size 1.27 1.27)) hide)
+    )
+    (property "LCSC Part" "C17557" (id 5) (at 269.24 243.84 0)
+      (effects (font (size 1.27 1.27)) hide)
+    )
     (pin "1")
     (pin "2")
@@
       (effects (font (size 1.27 1.27)) hide)
     )
+    (property "JLCPCB" "C17673" (id 4) (at 152.4 116.84 0)
+      (effects (font (size 1.27 1.27)) hide)
+    )
+    (property "LCSC Part" "C17673" (id 5) (at 152.4 116.84 0)
+      (effects (font (size 1.27 1.27)) hide)
+    )
     (pin "1")
     (pin "2")
@@
       (effects (font (size 1.27 1.27)) hide)
     )
+    (property "JLCPCB" "C17673" (id 4) (at 193.04 116.84 0)
+      (effects (font (size 1.27 1.27)) hide)
+    )
+    (property "LCSC Part" "C17673" (id 5) (at 193.04 116.84 0)
+      (effects (font (size 1.27 1.27)) hide)
+    )

Commit message: Update design.kicad_sch
Other:
- note added: "SMD DPDT: K3-2235S-K1 JS202011SCQN"
Changed lines of the file:
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@@
+    (effects (font (size 1.27 1.27)) (justify left bottom))
+  )
+  (text "SMD DPDT:\nK3-2235S-K1\nJS202011SCQN" (at 185.42 142.24 0)
     (effects (font (size 1.27 1.27)) (justify left bottom))
   )

Commit message: add Mfg Part #
Parts:
- C1, C2, C5, C6: MANUFACTURER_PART_NUMBER (none) -> CL21B105KBFNNNE
- C3, C7: MANUFACTURER_PART_NUMBER (none) -> CC0805KRX7R9BB104
- C4: MANUFACTURER_PART_NUMBER (none) -> CL21A106KAYNNNE
- C8: MANUFACTURER_PART_NUMBER (none) -> CL21A475KAQNNNE
- D1, D10, D3, D5, D9: MANUFACTURER_PART_NUMBER (none) -> NCD0805R1
- D2, D4, D6, D8: MANUFACTURER_PART_NUMBER (none) -> KT-0805G
- D7: MANUFACTURER_PART_NUMBER (none) -> SP0503BAHTG
- J14: MANUFACTURER_PART_NUMBER (none) -> BM04B-SRSS-TB(LF)(SN)
- J4: MANUFACTURER_PART_NUMBER (none) -> TYPE-C-31-M-12
- Q1, Q2: MANUFACTURER_PART_NUMBER (none) -> AO3400A
- R1, R2: MANUFACTURER_PART_NUMBER (none) -> C27834
- R10, R11, R15: MANUFACTURER_PART_NUMBER (none) -> 0805W8F4701T5E
- R12, R13, R14, R16, R17, R4, R6: MANUFACTURER_PART_NUMBER (none) -> 0805W8F2200T5E
- R3, R5, R7, R8: MANUFACTURER_PART_NUMBER (none) -> 0805W8F5600T5E
- R9: MANUFACTURER_PART_NUMBER (none) -> 0805W8F1001T5E
- SW1, SW2: MANUFACTURER_PART_NUMBER (none) -> K3-2235S-K1
- U1: MANUFACTURER_PART_NUMBER (none) -> ATTINY1616-SN
- U2: MANUFACTURER_PART_NUMBER (none) -> TPAP2112K-3.3TRG1
- U3: MANUFACTURER_PART_NUMBER (none) -> CP2105-F01-GMR
- U4: MANUFACTURER_PART_NUMBER (none) -> ATTINY1616-MNR
