File: design.kicad_sch (KiCad schematic)
At the start: 98 parts, among them J1 2601-3108, J10 Conn_01x04, J11 Conn_01x04, J12 Conn_01x03, J13 Conn_01x03, J14 BM04B-SRSS-TB_LF__SN_, J2 2601-3108, J3 2601-3108, J4 TYPE-C-31-M-12, J5 SKEDD-UPDI-4, J6 Conn_01x04, J7 Conn_01x04, J8 Conn_01x04, J9 Conn_01x04, Q1 AO3400A, Q2 AO3400A, SW1 K3-2235S-K1, SW2 K3-2235S-K1, U1 ATtiny1616-S, U2 AP2112K-3.3, U3 CP2105, U4 ATtiny1616-M

Commit message: update to v9
Parts:
- removed C6: 1uF 50V X7R ±10%, Capacitor_SMD:C_0805_2012Metric, symbol Device:C_Small
- removed C7: 100nF 50V X7R ±10%, Capacitor_SMD:C_0805_2012Metric, symbol Device:C_Small
- removed C8: 4.7uF 25V X5R ±10%, Capacitor_SMD:C_0805_2012Metric, symbol Device:C_Small
- removed D10, D9: Red, LED_SMD:LED_0805_2012Metric, symbol Device:LED_Small
- removed D8: Green, LED_SMD:LED_0805_2012Metric, symbol Device:LED_Small
- removed J12: Conn_01x03, Connector_PinHeader_2.54mm:PinHeader_1x03_P2.54mm_Vertical, symbol Connector_Generic:Conn_01x03
- removed JP5: CP-Bus, Jumper:SolderJumper-2_P1.3mm_Open_Pad1.0x1.5mm, symbol Jumper:SolderJumper_2_Open
- removed R10: 4.7k 1%, Resistor_SMD:R_0805_2012Metric, symbol Device:R_Small
- removed R12, R13, R14: 220 1%, Resistor_SMD:R_0805_2012Metric, symbol Device:R_Small
- removed R9: 1k 1%, Resistor_SMD:R_0805_2012Metric, symbol Device:R_Small
- removed SW2: K3-2235S-K1, Snapeda:easyeda2kicad_SW-SMD_K3-2235S-K1, symbol Snapeda:K3-2235S-K1
- removed U3: CP2105, Snapeda:CP2105_QFN24_0.5, symbol Snapeda:CP2105
- added U5: CH340K, Package_SO:SSOP-10-1EP_3.9x4.9mm_P1mm_EP2.1x3.3mm, symbol Interface_USB:CH340K
- C5: value 1uF 50V X7R ±10% -> 0.1uF 50V X7R ±10%
- gave numbers to parts that had none: 6
Connections:
- net V_CP2105 is gone; now on net VBUS: C5.1
- new net: U5.11 (GND), U5.3 (GND)
- no-connect marks 13 -> 4
Other:
- note removed: "PA1 TX_MCU PA2 RX_MCU"
- note removed: "SMD DPDT: K3-2235S-K1 JS202011SCQN"
- note removed: "close if slide switch not populated and programming only via the usb."
- moved on the sheet: C5

Commit message: Update design.kicad_sch
Parts:
- added C6: 0.1uF 50V X7R ±10%, Capacitor_SMD:C_0805_2012Metric, symbol Device:C_Small
- added U3: TS3USB30ERSWR, Package_DFN_QFN:UQFN-10_1.4x1.8mm_P0.4mm, symbol Interface_USB:TS3USB30ERSWR
Connections:
- net +3V3: now also U5.7 (VCC), C6.1, U3.9 (VCC)
- net D+: now also U5.1 (UD+)
- net D-: now also U5.2 (UD-)
- net GND: now also U5.11 (GND), U5.3 (GND), C6.2, U3.4 (GND), U3.8 (~{OE})
- net PB2: now also U3.6 (D2-)
- net PB3: now also U3.2 (D2+)
- net VBUS: now also U5.10 (V3)
- net at U5.4 (~{DTR}): now also U3.10 (S)
- net at U5.8 (TXD): now also U3.3 (D+)
- net at U5.9 (RXD): now also U3.5 (D-)
- no-connect marks 4 -> 6
Other:
- moved on the sheet: C5, U5

Commit message: allot
Parts:
- added R9: 560 1%, Resistor_SMD:R_0805_2012Metric, symbol Device:R_Small
Connections:
- net PA0: now also U3.7 (D1-), R9.2
- net at U3.1 (D1+): now also R9.1
Other:
- moved on the sheet: C6
